File: hardware/pcb/eval-board/eval-board.sch (KiCad schematic (older format))
At the start: 38 parts, among them J1 Conn_01x02, J2 Conn_01x24, J3 Conn_01x02, J4 Conn_01x02, J5 Conn_01x02, J6 Conn_01x02, J7 Conn_01x02, Q1 Si1308EDL, SW1 SW_SPDT, SW2 SW_SPST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

Commit message: etape intermediaire
Connections:
- net GND: now also J1.2 (Pin_2); no longer J1.1 (Pin_1)
- net at J3.1 (Pin_1): now also J1.1 (Pin_1); no longer J1.2 (Pin_2)
Changed lines of the file:
@@
 L Connector_Generic:Conn_01x02 J1
 U 1 1 61C3ECA6
-P 1000 1550
-F 0 "J1" H 918 1225 50  0000 C CNN
-F 1 "Conn_01x02" H 918 1316 50  0001 C CNN
-F 2 "Connector_PinHeader_2.54mm:PinHeader_1x02_P2.54mm_Vertical" H 1000 1550 50  0001 C CNN
-F 3 "~" H 1000 1550 50  0001 C CNN
-	1    1000 1550
-	-1   0    0    1
+P 1000 1450
+F 0 "J1" H 918 1125 50  0000 C CNN
+F 1 "Conn_01x02" H 918 1216 50  0001 C CNN
+F 2 "Connector_PinHeader_2.54mm:PinHeader_1x02_P2.54mm_Vertical" H 1000 1450 50  0001 C CNN
+F 3 "~" H 1000 1450 50  0001 C CNN
+	1    1000 1450
+	-1   0    0    -1
 $EndComp
 Wire Wire Line

Commit message: Carte eval finie
Parts:
- U3: footprint Package_DFN_QFN:DFN-6-1EP_2x2mm_P0.5mm_EP0.61x1.42mm -> Insa:uDFN-6-1EP_2x2mm_P0.65mm_EP1x1.6mm
Changed lines of the file:
@@
 encoding utf-8
 Sheet 1 1
-Title ""
-Date ""
-Rev ""
-Comp ""
+Title "EVAL-E.Ink"
+Date "2022-01-06"
+Rev "1.0"
+Comp "INSA - GEI"
 Comment1 ""
 Comment2 ""
@@
 F 0 "U3" H 2667 5615 50  0000 C CNN
 F 1 "MAX17220ELT" H 2667 5524 50  0000 C CNN
-F 2 "Package_DFN_QFN:DFN-6-1EP_2x2mm_P0.5mm_EP0.61x1.42mm" H 2600 5550 50  0001 C CNN
+F 2 "Insa:uDFN-6-1EP_2x2mm_P0.65mm_EP1x1.6mm" H 2600 5550 50  0001 C CNN
 F 3 "" H 2600 5550 50  0001 C CNN
 	1    2600 5050

Commit message: reorganisation de l'arborescence + renommage serveré
Parts:
- removed R3: R, Resistor_SMD:R_1206_3216Metric_Pad1.30x1.75mm_HandSolder, symbol Device:R
- added RV1: R_POT_TRIM, Potentiometer_SMD:Potentiometer_Bourns_3269P_Horizontal, symbol Device:R_POT_TRIM
- C1, C6, C7, C8: value 1µF -> 10µF
- C13, C14: footprint Capacitor_SMD:C_1206_3216Metric_Pad1.33x1.80mm_HandSolder -> Capacitor_SMD:C_0805_2012Metric_Pad1.18x1.45mm_HandSolder
- D1, D2, D3: footprint Diode_SMD:D_SOD-123 -> Diode_SMD:D_TUMD2
- L2: footprint Inductor_SMD:L_Wuerth_MAPI-1610 -> Inductor_SMD:L_Wuerth_MAPI-4030
Connections:
- net GND: now also RV1.2
- net at U3.4 (SEL): now also RV1.1
Changed lines of the file:
@@
 F 0 "D1" H 4000 2917 50  0000 C CNN
 F 1 "MBR0530" H 4000 2826 50  0000 C CNN
-F 2 "Diode_SMD:D_SOD-123" H 4000 2525 50  0001 C CNN
+F 2 "Diode_SMD:D_TUMD2" H 4000 2525 50  0001 C CNN
 F 3 "http://www.mccsemi.com/up_pdf/MBR0520~MBR0580(SOD123).pdf" H 4000 2700 50  0001 C CNN
 	1    4000 2700
@@
 F 0 "D2" V 4304 2780 50  0000 L CNN
 F 1 "MBR0530" V 4395 2780 50  0000 L CNN
-F 2 "Diode_SMD:D_SOD-123" H 4350 2525 50  0001 C CNN
+F 2 "Diode_SMD:D_TUMD2" H 4350 2525 50  0001 C CNN
 F 3 "http://www.mccsemi.com/up_pdf/MBR0520~MBR0580(SOD123).pdf" H 4350 2700 50  0001 C CNN
 	1    4350 2700
@@
 F 0 "D3" V 5046 2620 50  0000 R CNN
 F 1 "MBR0530" V 4955 2620 50  0000 R CNN
-F 2 "Diode_SMD:D_SOD-123" H 5000 2525 50  0001 C CNN
+F 2 "Diode_SMD:D_TUMD2" H 5000 2525 50  0001 C CNN
 F 3 "http://www.mccsemi.com/up_pdf/MBR0520~MBR0580(SOD123).pdf" H 5000 2700 50  0001 C CNN
 	1    5000 2700
@@
 P 8400 3500
 F 0 "C8" H 8515 3546 50  0000 L CNN
-F 1 "1µF" H 8515 3455 50  0000 L CNN
+F 1 "10µF" H 8515 3455 50  0000 L CNN
 F 2 "Capacitor_SMD:C_1206_3216Metric_Pad1.33x1.80mm_HandSolder" H 8438 3350 50  0001 C CNN
 F 3 "~" H 8400 3500 50  0001 C CNN
@@
 P 8000 3500
 F 0 "C7" H 8115 3546 50  0000 L CNN
-F 1 "1µF" H 8115 3455 50  0000 L CNN
+F 1 "10µF" H 8115 3455 50  0000 L CNN
 F 2 "Capacitor_SMD:C_1206_3216Metric_Pad1.33x1.80mm_HandSolder" H 8038 3350 50  0001 C CNN
 F 3 "~" H 8000 3500 50  0001 C CNN
@@
 P 7600 3500
 F 0 "C6" H 7715 3546 50  0000 L CNN
-F 1 "1µF" H 7715 3455 50  0000 L CNN
+F 1 "10µF" H 7715 3455 50  0000 L CNN
 F 2 "Capacitor_SMD:C_1206_3216Metric_Pad1.33x1.80mm_HandSolder" H 7638 3350 50  0001 C CNN
 F 3 "~" H 7600 3500 50  0001 C CNN
@@
 P 5550 3500
 F 0 "C1" H 5665 3546 50  0000 L CNN
-F 1 "1µF" H 5665 3455 50  0000 L CNN
+F 1 "10µF" H 5665 3455 50  0000 L CNN
 F 2 "Capacitor_SMD:C_1206_3216Metric_Pad1.33x1.80mm_HandSolder" H 5588 3350 50  0001 C CNN
 F 3 "~" H 5550 3500 50  0001 C CNN
@@
 F 0 "L2" H 2902 4046 50  0000 L CNN
 F 1 "2,2µH" H 2902 3955 50  0000 L CNN
-F 2 "Inductor_SMD:L_Wuerth_MAPI-1610" H 2850 4000 50  0001 C CNN
+F 2 "Inductor_SMD:L_Wuerth_MAPI-4030" H 2850 4000 50  0001 C CNN
 F 3 "~" H 2850 4000 50  0001 C CNN
 	1    2850 4000
@@
 F 0 "C13" H 1315 5246 50  0000 L CNN
 F 1 "10µF" H 1315 5155 50  0000 L CNN
-F 2 "Capacitor_SMD:C_1206_3216Metric_Pad1.33x1.80mm_HandSolder" H 1238 5050 50  0001 C CNN
+F 2 "Capacitor_SMD:C_0805_2012Metric_Pad1.18x1.45mm_HandSolder" H 1238 5050 50  0001 C CNN
 F 3 "~" H 1200 5200 50  0001 C CNN
 	1    1200 5200
@@
 F 0 "C14" H 3665 5346 50  0000 L CNN
 F 1 "10µF" H 3665 5255 50  0000 L CNN
-F 2 "Capacitor_SMD:C_1206_3216Metric_Pad1.33x1.80mm_HandSolder" H 3588 5150 50  0001 C CNN
+F 2 "Capacitor_SMD:C_0805_2012Metric_Pad1.18x1.45mm_HandSolder" H 3588 5150 50  0001 C CNN
 F 3 "~" H 3550 5300 50  0001 C CNN
 	1    3550 5300
 	1    0    0    -1
-$EndComp
-$Comp
-L Device:R R3
-U 1 1 61D861EB
-P 2050 5300
-F 0 "R3" V 2257 5300 50  0000 C CNN
-F 1 "R" V 2166 5300 50  0000 C CNN
-F 2 "Resistor_SMD:R_1206_3216Metric_Pad1.30x1.75mm_HandSolder" V 1980 5300 50  0001 C CNN
-F 3 "~" H 2050 5300 50  0001 C CNN
-	1    2050 5300
-	-1   0    0    1
 $EndComp
 $Comp
@@
 	1    0    0    -1
 $EndComp
-Wire Wire Line
-	2050 5550 2050 5450
 Wire Wire Line
 	1650 5600 1650 5550
@@
 	2050 3550 2050 4950
 Wire Wire Line
-	2200 5150 2050 5150
-Wire Wire Line
 	3000 5150 3000 5550
 Wire Wire Line
@@
 	7150 5300 7350 5300
 $Comp
-L power:+2V5 #PWR?
+L power:+2V5 #PWR0118
 U 1 1 6213A7B2
 P 6800 5850
-F 0 "#PWR?" H 6800 5700 50  0001 C CNN
+F 0 "#PWR0118" H 6800 5700 50  0001 C CNN
 F 1 "+2V5" H 6815 6023 50  0000 C CNN
 F 2 "" H 6800 5850 50  0001 C CNN
@@
 NoConn ~ 10300 5750
 NoConn ~ 10300 5850
+$Comp
+L Device:R_POT_TRIM RV1
+U 1 1 61DE5FE8
+P 1900 5300
+F 0 "RV1" H 1830 5346 50  0000 R CNN
+F 1 "R_POT_TRIM" H 1830 5255 50  0000 R CNN
+F 2 "Potentiometer_SMD:Potentiometer_Bourns_3269P_Horizontal" H 1900 5300 50  0001 C CNN
+F 3 "~" H 1900 5300 50  0001 C CNN
+	1    1900 5300
+	1    0    0    -1
+$EndComp
+Wire Wire Line
+	1900 5150 2200 5150
+Wire Wire Line
+	2050 5300 2050 5550
 $EndSCHEMATC
